File: usb-rs485.kicad_pcb (KiCad board)
At the start: 2 copper layers, 14.4 x 24.7 mm, 26 parts, among them IC1 THVD2450VDRCR, J1 USB4110GFA, U12 DF52-4S-0.8H(21), U9 CP2102N-A02-GQFN24R

Commit message: rename library to be for this
Parts:
- C20, C4, C5, C9: footprint robot-cortex:C_0603_1608Metric -> usb-rs485:C_0603_1608Metric
- C21, C8: footprint robot-cortex:C_0402_1005Metric -> usb-rs485:C_0402_1005Metric
- D1, D2, D3: footprint robot-cortex:D_SOD-923 -> usb-rs485:D_SOD-923
- D4, D5: footprint robot-cortex:LED_0603_1608Metric -> usb-rs485:LED_0603_1608Metric
- IC1: footprint robot-cortex:THVD2410VDRCR -> usb-rs485:THVD2410VDRCR
- J1: footprint robot-cortex:GCT_USB4110GFA -> usb-rs485:GCT_USB4110GFA
- J2, J3: footprint robot-cortex:ThruHoleBreadboardX4 -> usb-rs485:ThruHoleBreadboardX4
- R1, R19, R2, R3, R7, R8, R9: footprint robot-cortex:R_0402_1005Metric -> usb-rs485:R_0402_1005Metric
- U12: footprint robot-cortex:DF52-4S-0.8H(21) -> usb-rs485:DF52-4S-0.8H(21)
- U9: footprint robot-cortex:QFN50P400X400X80-25N -> usb-rs485:QFN50P400X400X80-25N
Changed lines of the file:
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@@
   (net 29 "unconnected-(U9-~{DSR}-Pad22)")
   (net 30 "unconnected-(U9-~{DCD}-Pad24)")
-  (footprint "robot-cortex:LED_0603_1608Metric" (layer "F.Cu")
+  (footprint "usb-rs485:LED_0603_1608Metric" (layer "F.Cu")
     (at 144.4225 106.895)
     (descr "LED SMD 0603 (1608 Metric), square (rectangular) end terminal, IPC_7351 nominal, (Body size source: http://www.tortai-tech.com/upload/download/2011102023233369053.pdf), generated with kicad-footprint-generator")
@@
     )
   )
-  (footprint "robot-cortex:R_0402_1005Metric" (layer "F.Cu")
+  (footprint "usb-rs485:R_0402_1005Metric" (layer "F.Cu")
     (at 139.15 99.39)
     (descr "Resistor SMD 0402 (1005 Metric), square (rectangular) end terminal, IPC_7351 nominal, (Body size source: IPC-SM-782 page 72, https://www.pcb-3d.com/wordpress/wp-content/uploads/ipc-sm-782a_amendment_1_and_2.pdf), generated with kicad-footprint-generator")
@@
     )
   )
-  (footprint "robot-cortex:QFN50P400X400X80-25N" (layer "F.Cu")
+  (footprint "usb-rs485:QFN50P400X400X80-25N" (layer "F.Cu")
     (at 143.11 103.27 -90)
     (property "A_MAX" "0.8")
@@
     )
   )
-  (footprint "robot-cortex:C_0402_1005Metric" (layer "F.Cu")
+  (footprint "usb-rs485:C_0402_1005Metric" (layer "F.Cu")
     (at 138.58 103.24 180)
     (descr "Capacitor SMD 0402 (1005 Metric), square (rectangular) end terminal, IPC_7351 nominal, (Body size source: IPC-SM-782 page 76, https://www.pcb-3d.com/wordpress/wp-content/uploads/ipc-sm-782a_amendment_1_and_2.pdf), generated with kicad-footprint-generator")
@@
     )
   )
-  (footprint "robot-cortex:DF52-4S-0.8H(21)" (layer "F.Cu")
+  (footprint "usb-rs485:DF52-4S-0.8H(21)" (layer "F.Cu")
     (at 143.11825 112.9465)
     (property "Sheetfile" "RS485-Transceiver.kicad_sch")
@@
     )
   )
-  (footprint "robot-cortex:R_0402_1005Metric" (layer "F.Cu")
+  (footprint "usb-rs485:R_0402_1005Metric" (layer "F.Cu")
     (at 143.104971 111.7915)
     (descr "Resistor SMD 0402 (1005 Metric), square (rectangular) end terminal, IPC_7351 nominal, (Body size source: IPC-SM-782 page 72, https://www.pcb-3d.com/wordpress/wp-content/uploads/ipc-sm-782a_amendment_1_and_2.pdf), generated with kicad-footprint-generator")
@@
     )
   )
-  (footprint "robot-cortex:D_SOD-923" (layer "F.Cu")
+  (footprint "usb-rs485:D_SOD-923" (layer "F.Cu")
     (at 143.89575 99.455 180)
     (descr "https://www.onsemi.com/pub/Collateral/ESD9B-D.PDF#page=4")
@@
     )
   )
-  (footprint "robot-cortex:C_0603_1608Metric" (layer "F.Cu")
+  (footprint "usb-rs485:C_0603_1608Metric" (layer "F.Cu")
     (at 146.16825 109.25 -90)
     (descr "Capacitor SMD 0603 (1608 Metric), square (rectangular) end terminal, IPC_7351 nominal, (Body size source: IPC-SM-782 page 76, https://www.pcb-3d.com/wordpress/wp-content/uploads/ipc-sm-782a_amendment_1_and_2.pdf), generated with kicad-footprint-generator")
@@
     )
   )
-  (footprint "robot-cortex:R_0402_1005Metric" (layer "F.Cu")
+  (footprint "usb-rs485:R_0402_1005Metric" (layer "F.Cu")
     (at 148.67825 99.745 90)
     (descr "Resistor SMD 0402 (1005 Metric), square (rectangular) end terminal, IPC_7351 nominal, (Body size source: IPC-SM-782 page 72, https://www.pcb-3d.com/wordpress/wp-content/uploads/ipc-sm-782a_amendment_1_and_2.pdf), generated with kicad-footprint-generator")
@@
     )
   )
-  (footprint "robot-cortex:R_0402_1005Metric" (layer "F.Cu")
+  (footprint "usb-rs485:R_0402_1005Metric" (layer "F.Cu")
     (at 137.52 99.39)
     (descr "Resistor SMD 0402 (1005 Metric), square (rectangular) end terminal, IPC_7351 nominal, (Body size source: IPC-SM-782 page 72, https://www.pcb-3d.com/wordpress/wp-content/uploads/ipc-sm-782a_amendment_1_and_2.pdf), generated with kicad-footprint-generator")
@@
     )
   )
-  (footprint "robot-cortex:GCT_USB4110GFA" (layer "F.Cu")
+  (footprint "usb-rs485:GCT_USB4110GFA" (layer "F.Cu")
     (at 143.11825 97.0375 180)
     (property "Availability" "In Stock")
@@
     )
   )
-  (footprint "robot-cortex:LED_0603_1608Metric" (layer "F.Cu")
+  (footprint "usb-rs485:LED_0603_1608Metric" (layer "F.Cu")
     (at 140.835 106.895 180)
     (descr "LED SMD 0603 (1608 Metric), square (rectangular) end terminal, IPC_7351 nominal, (Body size source: http://www.tortai-tech.com/upload/download/2011102023233369053.pdf), generated with kicad-footprint-generator")
@@
     )
   )
-  (footprint "robot-cortex:ThruHoleBreadboardX4" (layer "F.Cu")
+  (footprint "usb-rs485:ThruHoleBreadboardX4" (layer "F.Cu")
     (at 149.41825 107.99 90)
     (property "Sheetfile" "usb-rs485.kicad_sch")
@@
       (net 2 "GND") (pinfunction "4") (pintype "input"))
   )
-  (footprint "robot-cortex:THVD2410VDRCR" (layer "F.Cu")
+  (footprint "usb-rs485:THVD2410VDRCR" (layer "F.Cu")
     (at 142.868251 109.3915 -90)
     (property "Arrow Part Number" "")
@@
     )
   )
-  (footprint "robot-cortex:C_0402_1005Metric" (layer "F.Cu")
+  (footprint "usb-rs485:C_0402_1005Metric" (layer "F.Cu")
     (at 139.64 100.25 180)
     (descr "Capacitor SMD 0402 (1005 Metric), square (rectangular) end terminal, IPC_7351 nominal, (Body size source: IPC-SM-782 page 76, https://www.pcb-3d.com/wordpress/wp-content/uploads/ipc-sm-782a_amendment_1_and_2.pdf), generated with kicad-footprint-generator")
@@
     )
   )
-  (footprint "robot-cortex:C_0603_1608Metric" (layer "F.Cu")
+  (footprint "usb-rs485:C_0603_1608Metric" (layer "F.Cu")
     (at 146.26825 99.475)
     (descr "Capacitor SMD 0603 (1608 Metric), square (rectangular) end terminal, IPC_7351 nominal, (Body size source: IPC-SM-782 page 76, https://www.pcb-3d.com/wordpress/wp-content/uploads/ipc-sm-782a_amendment_1_and_2.pdf), generated with kicad-footprint-generator")
@@
     )
   )
-  (footprint "robot-cortex:D_SOD-923" (layer "F.Cu")
+  (footprint "usb-rs485:D_SOD-923" (layer "F.Cu")
     (at 142.32575 99.455)
     (descr "https://www.onsemi.com/pub/Collateral/ESD9B-D.PDF#page=4")
@@
     )
   )
-  (footprint "robot-cortex:R_0402_1005Metric" (layer "F.Cu")
+  (footprint "usb-rs485:R_0402_1005Metric" (layer "F.Cu")
     (at 140.22 103.8 -90)
     (descr "Resistor SMD 0402 (1005 Metric), square (rectangular) end terminal, IPC_7351 nominal, (Body size source: IPC-SM-782 page 72, https://www.pcb-3d.com/wordpress/wp-content/uploads/ipc-sm-782a_amendment_1_and_2.pdf), generated with kicad-footprint-generator")
@@
     )
   )
-  (footprint "robot-cortex:C_0603_1608Metric" (layer "F.Cu")
+  (footprint "usb-rs485:C_0603_1608Metric" (layer "F.Cu")
     (at 138.84175 102.18 180)
     (descr "Capacitor SMD 0603 (1608 Metric), square (rectangular) end terminal, IPC_7351 nominal, (Body size source: IPC-SM-782 page 76, https://www.pcb-3d.com/wordpress/wp-content/uploads/ipc-sm-782a_amendment_1_and_2.pdf), generated with kicad-footprint-generator")
@@
     )
   )
-  (footprint "robot-cortex:D_SOD-923" (layer "F.Cu")
+  (footprint "usb-rs485:D_SOD-923" (layer "F.Cu")
     (at 146.66825 100.5 180)
     (descr "https://www.onsemi.com/pub/Collateral/ESD9B-D.PDF#page=4")
@@
     )
   )
-  (footprint "robot-cortex:R_0402_1005Metric" (layer "F.Cu")
+  (footprint "usb-rs485:R_0402_1005Metric" (layer "F.Cu")
     (at 140.05825 108.26 90)
     (descr "Resistor SMD 0402 (1005 Metric), square (rectangular) end terminal, IPC_7351 nominal, (Body size source: IPC-SM-782 page 72, https://www.pcb-3d.com/wordpress/wp-content/uploads/ipc-sm-782a_amendment_1_and_2.pdf), generated with kicad-footprint-generator")
@@
     )
   )
-  (footprint "robot-cortex:R_0402_1005Metric" (layer "F.Cu")
+  (footprint "usb-rs485:R_0402_1005Metric" (layer "F.Cu")
     (at 146.16825 107.32 90)
     (descr "Resistor SMD 0402 (1005 Metric), square (rectangular) end terminal, IPC_7351 nominal, (Body size source: IPC-SM-782 page 72, https://www.pcb-3d.com/wordpress/wp-content/uploads/ipc-sm-782a_amendment_1_and_2.pdf), generated with kicad-footprint-generator")
@@
     )
   )
-  (footprint "robot-cortex:C_0603_1608Metric" (layer "F.Cu")
+  (footprint "usb-rs485:C_0603_1608Metric" (layer "F.Cu")
     (at 139.64 101.08 180)
     (descr "Capacitor SMD 0603 (1608 Metric), square (rectangular) end terminal, IPC_7351 nominal, (Body size source: IPC-SM-782 page 76, https://www.pcb-3d.com/wordpress/wp-content/uploads/ipc-sm-782a_amendment_1_and_2.pdf), generated with kicad-footprint-generator")
@@
     )
   )
-  (footprint "robot-cortex:ThruHoleBreadboardX4" (layer "F.Cu")
+  (footprint "usb-rs485:ThruHoleBreadboardX4" (layer "F.Cu")
     (at 136.91825 107.99 90)
     (property "Sheetfile" "usb-rs485.kicad_sch")
@@
   (gr_line (start 135.91825 92.24) (end 135.91825 114.44)
     (stroke (width 0.1) (type default)) (layer "Edge.Cuts"))
+  (gr_line (start 150.31825 92.24) (end 149.31825 91.24)
+    (stroke (width 0.1) (type default)) (layer "Edge.Cuts"))
   (gr_line (start 136.91825 91.24) (end 135.91825 92.24)
+    (stroke (width 0.1) (type default)) (layer "Edge.Cuts"))
+  (gr_line (start 148.81825 115.94) (end 150.31825 114.44)
     (stroke (width 0.1) (type default)) (layer "Edge.Cuts"))
   (gr_line (start 149.31825 91.24) (end 136.91825 91.24)
@@
   (gr_line (start 150.31825 114.44) (end 150.31825 92.24)
     (stroke (width 0.1) (type default)) (layer "Edge.Cuts"))
-  (gr_line (start 150.31825 92.24) (end 149.31825 91.24)
+  (gr_line (start 137.41825 115.94) (end 148.81825 115.94)
     (stroke (width 0.1) (type default)) (layer "Edge.Cuts"))
   (gr_line (start 135.91825 114.44) (end 137.41825 115.94)
     (stroke (width 0.1) (type default)) (layer "Edge.Cuts"))
-  (gr_line (start 137.41825 115.94) (end 148.81825 115.94)
-    (stroke (width 0.1) (type default)) (layer "Edge.Cuts"))
-  (gr_line (start 148.81825 115.94) (end 150.31825 114.44)
-    (stroke (width 0.1) (type default)) (layer "Edge.Cuts"))
   (gr_text "B" (at 137.81825 107.17 -90) (layer "B.SilkS")

Commit message: starting to add power
Parts:
- added C10: 10uF, usb-rs485:C_0603_1608Metric, F.Cu at (116.1, 105.5)
- added C11: 10uF, usb-rs485:C_0603_1608Metric, F.Cu at (116.1, 107.5)
- added C2: 4.7uF, usb-rs485:C_0603_1608Metric, F.Cu at (116.1, 99.8)
- added C3: 100nF, usb-rs485:C_0402_1005Metric, F.Cu at (122.9, 105.4)
- added C6: 10uF, usb-rs485:C_0603_1608Metric, F.Cu at (116.1, 101.8)
- added C7: 10uF, usb-rs485:C_0603_1608Metric, F.Cu at (116.1, 103.7)
- added L1: 1277AS-H-1R0M=P2, usb-rs485:L_1210_3225Metric, F.Cu at (119.9, 101.7)
- added R4: 470k, usb-rs485:R_0402_1005Metric, F.Cu at (127.1, 99.7)
- added R5: 150k, usb-rs485:R_0402_1005Metric, F.Cu at (127.1, 101.4)
- added R6: 100k, usb-rs485:C_0402_1005Metric, F.Cu at (122.9, 107.3)
- added U1: TPS63070, usb-rs485:VQFN-TPS63070, F.Cu at (119.7, 106.7)
