File: usb-rs485.kicad_pcb (KiCad board)
At the start: 4 copper layers, 14.5 x 24.7 mm, 37 parts, among them IC1 THVD2450VDRCR, J1 USB4110GFA, U1 TPS63070, U12 DF52-4S-0.8H(21), U9 CP2102N-A02-GQFN24R

Commit message: tweaks to layouts
Routing:
- net GND: vias 44 -> 46
Changed lines of the file:
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@@
   (via (at 148.00825 101.08) (size 0.45) (drill 0.2) (layers "F.Cu" "B.Cu") (net 2))
   (via (at 136.44825 93.58) (size 0.45) (drill 0.2) (layers "F.Cu" "B.Cu") (net 2))
+  (via (at 148.91825 115.04) (size 0.45) (drill 0.2) (layers "F.Cu" "B.Cu") (net 2))
   (via (at 141.61825 100.17) (size 0.45) (drill 0.2) (layers "F.Cu" "B.Cu") (net 2))
   (via (at 140.93825 106.14) (size 0.45) (drill 0.2) (layers "F.Cu" "B.Cu") (net 2))
-  (via (at 139.43825 114.08) (size 0.45) (drill 0.2) (layers "F.Cu" "B.Cu") (net 2))
-  (via (at 138.47825 114.05) (size 0.45) (drill 0.2) (layers "F.Cu" "B.Cu") (net 2))
+  (via (at 139.43825 114.04) (size 0.45) (drill 0.2) (layers "F.Cu" "B.Cu") (net 2))
+  (via (at 138.61825 114.05) (size 0.45) (drill 0.2) (layers "F.Cu" "B.Cu") (net 2))
   (via (at 147.005642 104.860913) (size 0.45) (drill 0.2) (layers "F.Cu" "B.Cu") (net 2))
   (via (at 136.35825 102.85) (size 0.45) (drill 0.2) (layers "F.Cu" "B.Cu") (net 2))
@@
   (via (at 140.81825 93.32) (size 0.45) (drill 0.2) (layers "F.Cu" "B.Cu") (net 2))
   (via (at 147.80825 102.5) (size 0.45) (drill 0.2) (layers "F.Cu" "B.Cu") (net 2))
-  (via (at 141.76825 115.42) (size 0.45) (drill 0.2) (layers "F.Cu" "B.Cu") (net 2))
+  (via (at 142.01825 115.54) (size 0.45) (drill 0.2) (layers "F.Cu" "B.Cu") (net 2))
   (via (at 146.99825 106.83) (size 0.45) (drill 0.2) (layers "F.Cu" "B.Cu") (net 2))
   (via (at 140.51825 109.34) (size 0.45) (drill 0.2) (layers "F.Cu" "B.Cu") (net 2))
@@
   (via (at 137.09825 102.33) (size 0.45) (drill 0.2) (layers "F.Cu" "B.Cu") (net 2))
   (via (at 137.91825 100.44) (size 0.45) (drill 0.2) (layers "F.Cu" "B.Cu") (net 2))
-  (via (at 143.22825 115.56) (size 0.45) (drill 0.2) (layers "F.Cu" "B.Cu") (net 2))
+  (via (at 143.21825 115.54) (size 0.45) (drill 0.2) (layers "F.Cu" "B.Cu") (net 2))
   (via (at 146.18825 95.44) (size 0.45) (drill 0.2) (layers "F.Cu" "B.Cu") (net 2))
-  (via (at 148.45825 113.42) (size 0.45) (drill 0.2) (layers "F.Cu" "B.Cu") (net 2))
+  (via (at 148.41825 113.44) (size 0.45) (drill 0.2) (layers "F.Cu" "B.Cu") (net 2))
   (via (at 137.21825 100.44) (size 0.45) (drill 0.2) (layers "F.Cu" "B.Cu") (net 2))
-  (via (at 149.10825 113.97) (size 0.45) (drill 0.2) (layers "F.Cu" "B.Cu") (net 2))
+  (via (at 149.91825 113.14) (size 0.45) (drill 0.2) (layers "F.Cu" "B.Cu") (net 2))
   (via (at 138.07825 105.44) (size 0.45) (drill 0.2) (layers "F.Cu" "B.Cu") (net 2))
   (via (at 136.41825 97.14) (size 0.45) (drill 0.2) (layers "F.Cu" "B.Cu") (net 2))
+  (via (at 144.51825 115.54) (size 0.45) (drill 0.2) (layers "F.Cu" "B.Cu") (net 2))
   (via (at 146.16825 93.16) (size 0.45) (drill 0.2) (layers "F.Cu" "B.Cu") (net 2))
   (via (at 149.664704 102.596398) (size 0.45) (drill 0.2) (layers "F.Cu" "B.Cu") (net 2))
@@
   (arc (start 142.81825 98.46) (mid 143.217909 97.861869) (end 143.35825 97.156325) (width 0.254) (layer "B.Cu") (net 4))
   (segment (start 144.404524 106.14) (end 144.59825 106.14) (width 0.254) (layer "F.Cu") (net 5))
+  (segment (start 147.01325 105.555) (end 147.44825 105.99) (width 0.254) (layer "F.Cu") (net 5))
+  (segment (start 147.83825 106.931543) (end 147.83825 107.24) (width 0.254) (layer "F.Cu") (net 5))
   (segment (start 145.383519 105.814731) (end 145.70825 105.49) (width 0.254) (layer "F.Cu") (net 5))
-  (segment (start 146.30825 105.39) (end 145.85825 104.94) (width 0.254) (layer "F.Cu") (net 5))
   (segment (start 145.85825 104.94) (end 145.85825 104.57) (width 0.254) (layer "F.Cu") (net 5))
   (segment (start 145.410261 104.02) (end 145.045 104.02) (width 0.254) (layer "F.Cu") (net 5))
   (segment (start 145.85825 104.57) (end 145.85825 104.79) (width 0.254) (layer "F.Cu") (net 5))
   (segment (start 143.368251 107.9915) (end 143.368251 107.641593) (width 0.254) (layer "F.Cu") (net 5))
+  (segment (start 146.08325 105.165) (end 146.18825 105.27) (width 0.254) (layer "F.Cu") (net 5))
   (segment (start 143.78473 106.53352) (end 144.01825 106.3) (width 0.254) (layer "F.Cu") (net 5))
   (segment (start 145.85825 105.127868) (end 145.85825 104.94) (width 0.254) (layer "F.Cu") (net 5))
-  (segment (start 149.41825 109.26) (end 148.149377 107.991127) (width 0.254) (layer "F.Cu") (net 5))
+  (segment (start 148.149377 107.991127) (end 149.41825 109.26) (width 0.254) (layer "F.Cu") (net 5))
+  (segment (start 146.477955 105.39) (end 146.614905 105.39) (width 0.254) (layer "F.Cu") (net 5))
+  (segment (start 145.85825 104.621802) (end 145.85825 104.425563) (width 0.254) (layer "F.Cu") (net 5))
   (segment (start 145.85825 104.57) (end 145.85825 104.425563) (width 0.254) (layer "F.Cu") (net 5))
-  (segment (start 147.44825 105.99) (end 146.84825 105.39) (width 0.254) (layer "F.Cu") (net 5))
   (segment (start 145.85825 104.94) (end 145.85825 104.425563) (width 0.254) (layer "F.Cu") (net 5))
-  (segment (start 146.84825 105.39) (end 146.30825 105.39) (width 0.254) (layer "F.Cu") (net 5))
-  (segment (start 147.83825 107.24) (end 147.83825 106.931543) (width 0.254) (layer "F.Cu") (net 5))
   (arc (start 145.85825 104.425563) (mid 145.829662 104.281842) (end 145.74825 104.16) (width 0.254) (layer "F.Cu") (net 5))
+  (arc (start 147.83825 107.24) (mid 147.91911 107.646507) (end 148.149377 107.991127) (width 0.254) (layer "F.Cu") (net 5))
   (arc (start 143.635 106.895) (mid 143.673914 106.699368) (end 143.78473 106.53352) (width 0.254) (layer "F.Cu") (net 5))
   (arc (start 144.59825 106.14) (mid 145.023234 106.055465) (end 145.383519 105.814731) (width 0.254) (layer "F.Cu") (net 5))
+  (arc (start 146.18825 105.27) (mid 146.321168 105.358813) (end 146.477955 105.39) (width 0.254) (layer "F.Cu") (net 5))
   (arc (start 143.368251 107.641593) (mid 143.448622 107.23754) (end 143.6775 106.895) (width 0.254) (layer "F.Cu") (net 5))
-  (arc (start 147.83825 106.931543) (mid 147.736892 106.421983) (end 147.44825 105.99) (width 0.254) (layer "F.Cu") (net 5))
-  (arc (start 148.149377 107.991127) (mid 147.91911 107.646507) (end 147.83825 107.24) (width 0.254) (layer "F.Cu") (net 5))
+  (arc (start 147.44825 105.99) (mid 147.736892 106.421983) (end 147.83825 106.931543) (width 0.254) (layer "F.Cu") (net 5))
   (arc (start 145.74825 104.16) (mid 145.59318 104.056385) (end 145.410261 104.02) (width 0.254) (layer "F.Cu") (net 5))
+  (arc (start 146.08325 105.165) (mid 145.916726 104.915779) (end 145.85825 104.621802) (width 0.254) (layer "F.Cu") (net 5))
   (arc (start 145.70825 105.49) (mid 145.819266 105.323853) (end 145.85825 105.127868) (width 0.254) (layer "F.Cu") (net 5))
   (arc (start 144.01825 106.3) (mid 144.195474 106.181583) (end 144.404524 106.14) (width 0.254) (layer "F.Cu") (net 5))
+  (arc (start 146.614905 105.39) (mid 146.830487 105.432882) (end 147.01325 105.555) (width 0.254) (layer "F.Cu") (net 5))
   (segment (start 146.01325 106.88236) (end 145.240515 106.88236) (width 0.254) (layer "F.Cu") (net 6))
   (arc (start 145.240515 106.88236) (mid 145.224001 106.885645) (end 145.21 106.895) (width 0.254) (layer "F.Cu") (net 6))
@@
   (via (at 141.15825 112.51) (size 0.45) (drill 0.2) (layers "F.Cu" "B.Cu") (net 36))
   (arc (start 141.91825 112.9465) (mid 141.619375 112.88705) (end 141.366001 112.717751) (width 0.381) (layer "F.Cu") (net 36))
-  (segment (start 138.20825 114.82) (end 137.73225 114.344) (width 0.381) (layer "In1.Cu") (net 36))
-  (segment (start 140.207123 114.651127) (end 140.08825 114.77) (width 0.381) (layer "In1.Cu") (net 36))
-  (segment (start 146.75825 115.07) (end 146.02825 114.34) (width 0.381) (layer "In1.Cu") (net 36))
-  (segment (start 137.73225 114.344) (end 136.91825 114.344) (width 0.381) (layer "In1.Cu") (net 36))
-  (segment (start 139.96754 114.82) (end 138.20825 114.82) (width 0.381) (layer "In1.Cu") (net 36))
-  (segment (start 146.02825 114.34) (end 140.95825 114.34) (width 0.381) (layer "In1.Cu") (net 36))
-  (arc (start 140.95825 114.34) (mid 140.551743 114.420859) (end 140.207123 114.651127) (width 0.381) (layer "In1.Cu") (net 36))
-  (arc (start 140.08825 114.77) (mid 140.032868 114.807005) (end 139.96754 114.82) (width 0.381) (layer "In1.Cu") (net 36))
+  (segment (start 141.221803 114.34) (end 144.995875 114.34) (width 0.381) (layer "In1.Cu") (net 36))
+  (segment (start 138.469879 114.82) (end 140.062981 114.82) (width 0.381) (layer "In1.Cu") (net 36))
+  (segment (start 136.91825 114.344) (end 137.320714 114.344) (width 0.381) (layer "In1.Cu") (net 36))
+  (arc (start 140.062981 114.82) (mid 140.363491 114.760225) (end 140.61825 114.59) (width 0.381) (layer "In1.Cu") (net 36))
+  (arc (start 137.320714 114.344) (mid 137.700924 114.419628) (end 138.02325 114.635) (width 0.381) (layer "In1.Cu") (net 36))
+  (arc (start 138.02325 114.635) (mid 138.228165 114.77192) (end 138.469879 114.82) (width 0.381) (layer "In1.Cu") (net 36))
+  (arc (start 144.995875 114.34) (mid 145.949665 114.529721) (end 146.75825 115.07) (width 0.381) (layer "In1.Cu") (net 36))
+  (arc (start 140.61825 114.59) (mid 140.895162 114.404973) (end 141.221803 114.34) (width 0.381) (layer "In1.Cu") (net 36))
   (segment (start 146.12825 114.84) (end 146.202981 114.84) (width 0.381) (layer "B.Cu") (net 36))
   (segment (start 141.260677 112.467574) (end 141.72825 112) (width 0.381) (layer "B.Cu") (net 36))
@@
         (xy 140.05825 113.29)
         (xy 140.05825 113.49)
-        (xy 137.908225 113.493147)
-        (xy 137.678865 113.679998)
+        (xy 138.55338 113.492203)
+        (xy 137.680686 114.203154)
         (xy 137.688282 116.386069)
-        (xy 135.66825 116.36)
-        (xy 135.68825 112.59)
-        (xy 138.438205 112.598009)
-        (xy 139.40325 111.645)
+        (xy 135.68825 116.39)
+        (xy 135.68825 112.64)
+        (xy 137.138205 112.64)
+        (xy 138.10325 111.645)
         (xy 142.26825 111.645)
         (xy 142.59325 111.97)

Commit message: lights
Parts:
- added D6: 150060GS84000, usb-rs485:LED_0603_1608Metric, B.Cu at (138.8, 114.4)
- added R10: 470, usb-rs485:R_0402_1005Metric, B.Cu at (140.2, 115.4)
Routing:
- net Net-(D6-K): track 0.00 -> 1.08 mm
- net GND: vias 46 -> 49
Changed lines of the file:
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@@
   (net 35 "Net-(U1-PG)")
   (net 36 "/7V0")
+  (net 37 "Net-(D6-K)")
   (footprint "usb-rs485:LED_0603_1608Metric" (layer "F.Cu")
     (at 144.4225 106.895)
@@
     )
   )
+  (footprint "usb-rs485:LED_0603_1608Metric" (layer "B.Cu")
+    (at 138.83825 114.41 90)
+    (descr "LED SMD 0603 (1608 Metric), square (rectangular) end terminal, IPC_7351 nominal, (Body size source: http://www.tortai-tech.com/upload/download/2011102023233369053.pdf), generated with kicad-footprint-generator")
+    (tags "LED")
+    (property "Sheetfile" "usb-rs485.kicad_sch")
+    (property "Sheetname" "")
+    (property "ki_description" "Light emitting diode")
+    (property "ki_keywords" "LED diode")
+    (attr smd)
+    (fp_text reference "D6" (at 0 1.43) (layer "B.SilkS") hide
+        (effects (font (size 1 1) (thickness 0.15)) (justify mirror))
+    )
+    (fp_text value "150060GS84000" (at 0 -1.43 90) (layer "B.Fab")
+        (effects (font (size 1 1) (thickness 0.15)) (justify mirror))
+    )
+    (fp_text user "${REFERENCE}" (at 0 0 90) (layer "B.Fab")
+        (effects (font (size 0.4 0.4) (thickness 0.06)) (justify mirror))
+    )
+    (fp_line (start -1.485 -0.735) (end 0.8 -0.735)
+      (stroke (width 0.12) (type solid)) (layer "B.SilkS"))
+    (fp_line (start -1.485 0.735) (end -1.485 -0.735)
+      (stroke (width 0.12) (type solid)) (layer "B.SilkS"))
+    (fp_line (start 0.8 0.735) (end -1.485 0.735)
+      (stroke (width 0.12) (type solid)) (layer "B.SilkS"))
+    (fp_rect (start -1.2 0.5) (end 1.2 -0.475)
+      (stroke (width 0.12) (type default)) (fill none) (layer "B.CrtYd"))
+    (fp_line (start -0.8 -0.4) (end 0.8 -0.4)
+      (stroke (width 0.1) (type solid)) (layer "B.Fab"))
+    (fp_line (start -0.8 0.1) (end -0.8 -0.4)
+      (stroke (width 0.1) (type solid)) (layer "B.Fab"))
+    (fp_line (start -0.5 0.4) (end -0.8 0.1)
+      (stroke (width 0.1) (type solid)) (layer "B.Fab"))
+    (fp_line (start 0.8 -0.4) (end 0.8 0.4)
+      (stroke (width 0.1) (type solid)) (layer "B.Fab"))
+    (fp_line (start 0.8 0.4) (end -0.5 0.4)
+      (stroke (width 0.1) (type solid)) (layer "B.Fab"))
+    (pad "1" smd roundrect (at -0.7875 0 90) (size 0.875 0.95) (layers "B.Cu" "B.Paste" "B.Mask") (roundrect_rratio 0.25)
+      (net 37 "Net-(D6-K)") (pinfunction "K") (pintype "passive"))
+    (pad "2" smd roundrect (at 0.7875 0 90) (size 0.875 0.95) (layers "B.Cu" "B.Paste" "B.Mask") (roundrect_rratio 0.25)
+      (net 36 "/7V0") (pinfunction "A") (pintype "passive"))
+    (model "${KIPRJMOD}/3dModels/LED_0603_1608Metric.step"
+      (offset (xyz 0 0 0))
+      (scale (xyz 1 1 1))
+      (rotate (xyz 0 0 0))
+    )
+  )
   (footprint "usb-rs485:C_0603_1608Metric" (layer "B.Cu")
     (at 140.64825 111.29 90)
@@
       (net 2 "GND") (pintype "passive") (solder_mask_margin 0.0508))
     (model "${KIPRJMOD}/3dModels/C_0603_1608Metric.step"
+      (offset (xyz 0 0 0))
+      (scale (xyz 1 1 1))
+      (rotate (xyz 0 0 0))
+    )
+  )
+  (footprint "usb-rs485:R_0402_1005Metric" (layer "B.Cu")
+    (at 140.22825 115.43 180)
+    (descr "Resistor SMD 0402 (1005 Metric), square (rectangular) end terminal, IPC_7351 nominal, (Body size source: IPC-SM-782 page 72, https://www.pcb-3d.com/wordpress/wp-content/uploads/ipc-sm-782a_amendment_1_and_2.pdf), generated with kicad-footprint-generator")
+    (tags "resistor")
+    (property "Sheetfile" "usb-rs485.kicad_sch")
+    (property "Sheetname" "")
+    (property "ki_description" "Resistor, US symbol")
+    (property "ki_keywords" "R res resistor")
+    (attr smd)
+    (fp_text reference "R10" (at 2.95 1.45) (layer "B.CrtYd") hide
+        (effects (font (size 1 1) (thickness 0.15)) (justify mirror))
+    )
+    (fp_text value "470" (at 0 -1.17) (layer "B.Fab") hide
+        (effects (font (size 1 1) (thickness 0.15)) (justify mirror))
+    )
+    (fp_text user "${REFERENCE}" (at 0 0) (layer "B.Fab")
+        (effects (font (size 0.26 0.26) (thickness 0.04)) (justify mirror))
+    )
+    (fp_line (start -0.475 0) (end -0.475 -0.225)
+      (stroke (width 0.12) (type default)) (layer "B.CrtYd"))
+    (fp_line (start -0.475 0) (end -0.475 0.225)
+      (stroke (width 0.12) (type default)) (layer "B.CrtYd"))
+    (fp_line (start 0 -0.225) (end -0.475 -0.225)
+      (stroke (width 0.12) (type default)) (layer "B.CrtYd"))
+    (fp_line (start 0 -0.225) (end 0.475 -0.225)
+      (stroke (width 0.12) (type default)) (layer "B.CrtYd"))
+    (fp_line (start 0 0.225) (end -0.475 0.225)
+      (stroke (width 0.12) (type default)) (layer "B.CrtYd"))
+    (fp_line (start 0 0.225) (end 0.475 0.225)
+      (stroke (width 0.12) (type default)) (layer "B.CrtYd"))
+    (fp_line (start 0.475 0) (end 0.475 -0.225)
+      (stroke (width 0.12) (type default)) (layer "B.CrtYd"))
+    (fp_line (start 0.475 0) (end 0.475 0.225)
+      (stroke (width 0.12) (type default)) (layer "B.CrtYd"))
+    (fp_line (start -0.525 -0.27) (end -0.525 0.27)
+      (stroke (width 0.1) (type solid)) (layer "B.Fab"))
+    (fp_line (start -0.525 0.27) (end 0.525 0.27)
+      (stroke (width 0.1) (type solid)) (layer "B.Fab"))
+    (fp_line (start 0.525 -0.27) (end -0.525 -0.27)
+      (stroke (width 0.1) (type solid)) (layer "B.Fab"))
+    (fp_line (start 0.525 0.27) (end 0.525 -0.27)
+      (stroke (width 0.1) (type solid)) (layer "B.Fab"))
+    (pad "1" smd roundrect (at -0.375 0 180) (size 0.45 0.5) (layers "B.Cu" "B.Paste" "B.Mask") (roundrect_rratio 0.25)
+      (net 2 "GND") (pintype "passive") (solder_mask_margin 0.0508))
+    (pad "2" smd roundrect (at 0.375 0 180) (size 0.45 0.5) (layers "B.Cu" "B.Paste" "B.Mask") (roundrect_rratio 0.25)
+      (net 37 "Net-(D6-K)") (pintype "passive") (solder_mask_margin 0.0508))
+    (model "${KICAD6_3DMODEL_DIR}/Resistor_SMD.3dshapes/R_0402_1005Metric.wrl"
       (offset (xyz 0 0 0))
       (scale (xyz 1 1 1))
@@
   (via (at 141.61825 100.17) (size 0.45) (drill 0.2) (layers "F.Cu" "B.Cu") (net 2))
   (via (at 140.93825 106.14) (size 0.45) (drill 0.2) (layers "F.Cu" "B.Cu") (net 2))
-  (via (at 139.43825 114.04) (size 0.45) (drill 0.2) (layers "F.Cu" "B.Cu") (net 2))
-  (via (at 138.61825 114.05) (size 0.45) (drill 0.2) (layers "F.Cu" "B.Cu") (net 2))
+  (via (at 136.17825 113.11) (size 0.45) (drill 0.2) (layers "F.Cu" "B.Cu") (net 2))
+  (via (at 136.28825 110.55) (size 0.45) (drill 0.2) (layers "F.Cu" "B.Cu") (net 2))
   (via (at 147.005642 104.860913) (size 0.45) (drill 0.2) (layers "F.Cu" "B.Cu") (net 2))
   (via (at 136.35825 102.85) (size 0.45) (drill 0.2) (layers "F.Cu" "B.Cu") (net 2))
@@
   (via (at 140.51825 109.34) (size 0.45) (drill 0.2) (layers "F.Cu" "B.Cu") (net 2))
   (via (at 139.71825 105.99) (size 0.45) (drill 0.2) (layers "F.Cu" "B.Cu") (net 2))
+  (via (at 149.96825 110.58) (size 0.45) (drill 0.2) (layers "F.Cu" "B.Cu") (net 2))
   (via (at 146.21825 102.8) (size 0.45) (drill 0.2) (layers "F.Cu" "B.Cu") (net 2))
   (via (at 149.60825 101.06) (size 0.45) (drill 0.2) (layers "F.Cu" "B.Cu") (net 2))
@@
   (via (at 137.21825 100.44) (size 0.45) (drill 0.2) (layers "F.Cu" "B.Cu") (net 2))
   (via (at 149.91825 113.14) (size 0.45) (drill 0.2) (layers "F.Cu" "B.Cu") (net 2))
+  (via (at 139.60825 111.7074) (size 0.45) (drill 0.2) (layers "F.Cu" "B.Cu") (net 2))
   (via (at 138.07825 105.44) (size 0.45) (drill 0.2) (layers "F.Cu" "B.Cu") (net 2))
   (via (at 136.41825 97.14) (size 0.45) (drill 0.2) (layers "F.Cu" "B.Cu") (net 2))
@@
   (via (at 145.04825 105.21) (size 0.45) (drill 0.2) (layers "F.Cu" "B.Cu") (net 2))
   (via (at 145.59825 101.19) (size 0.45) (drill 0.2) (layers "F.Cu" "B.Cu") (net 2))
+  (via (at 149.95825 107.92) (size 0.45) (drill 0.2) (layers "F.Cu" "B.Cu") (net 2))
   (segment (start 142.86 101.335) (end 142.86825 101.32675) (width 0.254) (layer "F.Cu") (net 3))
   (segment (start 143.91025 96.901246) (end 143.91025 97.38305) (width 0.254) (layer "F.Cu") (net 3))
@@
   (arc (start 141.15825 112.51) (mid 141.156412 112.519239) (end 141.151179 112.527071) (width 0.381) (layer "B.Cu") (net 36))
   (arc (start 141.15825 112.51) (mid 141.213683 112.498974) (end 141.260677 112.467574) (width 0.381) (layer "B.Cu") (net 36))
+  (segment (start 138.931215 115.1975) (end 138.83825 115.1975) (width 0.381) (layer "B.Cu") (net 37))
+  (segment (start 139.85325 115.43) (end 139.496123 115.43) (width 0.381) (layer "B.Cu") (net 37))
+  (segment (start 139.056261 115.322546) (end 138.931215 115.1975) (width 0.381) (layer "B.Cu") (net 37))
+  (arc (start 139.496123 115.43) (mid 139.270057 115.402124) (end 139.056261 115.322546) (width 0.381) (layer "B.Cu") (net 37))
   (zone (net 1) (net_name "+3V3") (layer "F.Cu") (hatch edge 0.5)
     (priority 3)
