File: PSU_TPS63070RNMR.kicad_sch (KiCad schematic)
At the start: 9 parts, among them U1 TPS63070

Commit message: wiring in boost to 6V
Connections:
- net L1: now reaches L1.1, U1.11 (L1)
- net L2: now reaches L1.2, U1.9 (L2)
Changed lines of the file:
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@@
   (junction (at 135.89 95.885) (diameter 0) (color 0 0 0 0)
+  )
+  (junction (at 137.795 64.77) (diameter 0) (color 0 0 0 0)
+  )
+  (junction (at 113.03 64.77) (diameter 0) (color 0 0 0 0)
   )
   (junction (at 164.465 78.105) (diameter 0) (color 0 0 0 0)
@@
     (stroke (width 0) (type default))
   )
+  (wire (pts (xy 137.795 63.5) (xy 137.795 64.77))
+    (stroke (width 0) (type default))
+  )
   (wire (pts (xy 135.89 93.345) (xy 135.89 95.885))
     (stroke (width 0) (type default))
@@
   )
   (wire (pts (xy 112.395 92.075) (xy 115.57 92.075))
+    (stroke (width 0) (type default))
+  )
+  (wire (pts (xy 113.03 63.5) (xy 113.03 64.77))
     (stroke (width 0) (type default))
   )
@@
     (effects (font (size 1.27 1.27)) (justify left bottom))
   )
+  (label "L1" (at 113.03 63.5 180) (fields_autoplaced)
+    (effects (font (size 1.27 1.27)) (justify right bottom))
+  )
+  (label "L2" (at 137.795 63.5 0) (fields_autoplaced)
+    (effects (font (size 1.27 1.27)) (justify left bottom))
+  )
