File: RS485-Transceiver.kicad_sch (KiCad schematic)
At the start: 5 parts, among them IC1 THVD2450VDRCR, U12 DF52-4S-0.8H(21)

Commit message: backups removalled schematic looking correct if not good
Connections:
- net VBAT is gone; now on net 5V0: U12.1
Changed lines of the file:
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@@
-    (stroke (width 0) (type default))
-  )
-  (wire (pts (xy 55.88 104.14) (xy 52.07 104.14))
     (stroke (width 0) (type default))
   )
@@
     (effects (font (size 1.27 1.27)) (justify left bottom))
   )
-  (label "VBAT" (at 55.88 104.14 0) (fields_autoplaced)
-    (effects (font (size 1.27 1.27)) (justify left bottom))
-  )
   (label "UART_DE" (at 56.515 97.79 0) (fields_autoplaced)
     (effects (font (size 1.27 1.27)) (justify left bottom))
@@
     (effects (font (size 1.27 1.27)) (justify left bottom))
   )
-  (label "VBAT" (at 160.655 83.185 180) (fields_autoplaced)
-    (effects (font (size 1.27 1.27)) (justify right bottom))
-  )
   (label "UART_TX" (at 56.515 93.345 0) (fields_autoplaced)
     (effects (font (size 1.27 1.27)) (justify left bottom))
   )
+  (label "+5V0" (at 160.655 83.185 180) (fields_autoplaced)
+    (effects (font (size 1.27 1.27)) (justify right bottom))
+  )
   (hierarchical_label "UART_TX" (shape input) (at 52.07 93.345 180) (fields_autoplaced)
     (effects (font (size 1.27 1.27)) (justify right))
@@
   )
   (hierarchical_label "GND" (shape input) (at 52.07 84.455 180) (fields_autoplaced)
-    (effects (font (size 1.27 1.27)) (justify right))
-  )
-  (hierarchical_label "VBAT" (shape input) (at 52.07 104.14 180) (fields_autoplaced)
     (effects (font (size 1.27 1.27)) (justify right))
   )
@@
   (symbol (lib_id "robot-cortex:R") (at 142.875 93.345 0) (mirror x) (unit 1)
     (in_bom yes) (on_board yes) (dnp no)
-    (property "Reference" "R19" (at 138.938 93.98 0)
+    (property "Reference" "R19" (at 144.145 92.075 0)
       (effects (font (size 1.27 1.27)) (justify left))
     )
-    (property "Value" "120" (at 145.923 93.98 0)
-      (effects (font (size 1.27 1.27)))
-    )
+    (property "Value" "120" (at 146.05 94.615 0)
+      (effects (font (size 1.27 1.27)))
+    )

Commit message: library table
Parts:
- C1, C28: symbol Device:C -> usb-rs485:C
- IC1: symbol robot-cortex:THVD2450VDRCR -> usb-rs485:THVD2450VDRCR
- R19: symbol robot-cortex:R -> usb-rs485:R
- U12: symbol foc-pcb:DF52-4S-0.8H(21) -> usb-rs485:DF52-4S-0.8H(21)
Changed lines of the file:
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@@
     (effects (font (size 1.27 1.27)) (justify right))
   )
-  (symbol (lib_id "robot-cortex:THVD2450VDRCR") (at 103.505 89.535 0) (unit 1)
+  (symbol (lib_id "usb-rs485:THVD2450VDRCR") (at 103.505 89.535 0) (unit 1)
     (in_bom yes) (on_board yes) (dnp no) (fields_autoplaced)
     (property "Reference" "IC1" (at 118.3991 111.76 0)
@@
     )
   )
-  (symbol (lib_id "foc-pcb:DF52-4S-0.8H(21)") (at 167.005 93.345 0) (unit 1)
+  (symbol (lib_id "usb-rs485:DF52-4S-0.8H(21)") (at 167.005 93.345 0) (unit 1)
     (in_bom yes) (on_board yes) (dnp no)
     (property "Reference" "U12" (at 166.37 81.915 0)
@@
     )
   )
-  (symbol (lib_id "Device:C") (at 100.965 77.47 0) (unit 1)
+  (symbol (lib_id "usb-rs485:C") (at 100.965 77.47 0) (unit 1)
     (in_bom yes) (on_board yes) (dnp no) (fields_autoplaced)
     (property "Reference" "C1" (at 104.902 76.2 0)
@@
     )
   )
-  (symbol (lib_id "robot-cortex:R") (at 142.875 93.345 0) (mirror x) (unit 1)
+  (symbol (lib_id "usb-rs485:R") (at 142.875 93.345 0) (mirror x) (unit 1)
     (in_bom yes) (on_board yes) (dnp no)
     (property "Reference" "R19" (at 144.145 92.075 0)
@@
     )
   )
-  (symbol (lib_id "Device:C") (at 129.54 82.55 0) (unit 1)
+  (symbol (lib_id "usb-rs485:C") (at 129.54 82.55 0) (unit 1)
     (in_bom yes) (on_board yes) (dnp no) (fields_autoplaced)
     (property "Reference" "C28" (at 133.477 81.28 0)

Commit message: routing
Parts:
- added C9: 10uF 0603, robot-cortex:C_0603_1608Metric, symbol usb-rs485:Capacitor
Connections:
- net +3V3: now also C9.1
- net GND: now also C9.2
Changed lines of the file:
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@@
+    (stroke (width 0) (type default))
+  )
+  (wire (pts (xy 149.86 59.055) (xy 149.86 58.42))
     (stroke (width 0) (type default))
   )
@@
     )
   )
+  (symbol (lib_id "power:GND") (at 149.86 66.675 0) (mirror y) (unit 1)
+    (in_bom yes) (on_board yes) (dnp no) (fields_autoplaced)
+    (property "Reference" "#PWR06" (at 149.86 73.025 0)
+      (effects (font (size 1.27 1.27)) hide)
+    )
+    (property "Value" "GND" (at 149.86 71.755 0)
+      (effects (font (size 1.27 1.27)))
+    )
+    (property "Footprint" "" (at 149.86 66.675 0)
+      (effects (font (size 1.27 1.27)) hide)
+    )
+    (property "Datasheet" "" (at 149.86 66.675 0)
+      (effects (font (size 1.27 1.27)) hide)
+    )
+    (pin "1")
+    (instances
+      (project "usb-rs485"
+        (path "/19e4cb9f-d0a4-4ce0-8aa4-5fe95563dc37/c6177953-2b5d-4464-aaa8-66a87e9974f4"
+          (reference "#PWR06") (unit 1)
+        )
+      )
+    )
+  )
+  (symbol (lib_id "usb-rs485:Capacitor") (at 149.86 62.865 0) (mirror y) (unit 1)
+    (in_bom yes) (on_board yes) (dnp no)
+    (property "Reference" "C9" (at 149.225 60.96 0)
+      (effects (font (size 1.27 1.27)) (justify left))
+    )
+    (property "Value" "10uF 0603" (at 145.415 67.945 90)
+      (effects (font (size 1.27 1.27)) (justify left))
+    )
+    (property "Footprint" "robot-cortex:C_0603_1608Metric" (at 148.8948 66.675 0)
+      (effects (font (size 1.27 1.27)) hide)
+    )
+    (property "Datasheet" "~" (at 149.86 62.865 0)
+      (effects (font (size 1.27 1.27)) hide)
+    )
+    (property "Voltage" "10V" (at 124.46 66.675 90)
+      (effects (font (size 1.27 1.27)) (justify left) hide)
+    )
+    (pin "1")
+    (pin "2")
+    (instances
+      (project "usb-rs485"
+        (path "/19e4cb9f-d0a4-4ce0-8aa4-5fe95563dc37/c6177953-2b5d-4464-aaa8-66a87e9974f4"
+          (reference "C9") (unit 1)
+        )
+      )
+    )
+  )
   (symbol (lib_id "power:GND") (at 129.54 78.74 0) (mirror x) (unit 1)
     (in_bom yes) (on_board yes) (dnp no) (fields_autoplaced)
@@
         )
       )
+    )
+  )
+  (symbol (lib_id "power:+3V3") (at 149.86 58.42 0) (mirror y) (unit 1)
+    (in_bom yes) (on_board yes) (dnp no)
+    (property "Reference" "#PWR03" (at 149.86 62.23 0)
+      (effects (font (size 1.27 1.27)) hide)
+    )
+    (property "Value" "+3V3" (at 153.67 57.15 0)
+      (effects (font (size 1.27 1.27)))
+    )
+    (property "Footprint" "" (at 149.86 58.42 0)
+      (effects (font (size 1.27 1.27)) hide)
+    )
+    (property "Datasheet" "" (at 149.86 58.42 0)
+      (effects (font (size 1.27 1.27)) hide)
+    )
+    (pin "1")
+    (instances
+      (project "usb-rs485"
+        (path "/19e4cb9f-d0a4-4ce0-8aa4-5fe95563dc37/c6177953-2b5d-4464-aaa8-66a87e9974f4"
+          (reference "#PWR03") (unit 1)
+        )
+      )

Commit message: routed, thru holes. ready to order i think
Connections:
- net RS1_A renamed RS485-A
- net RS1_B renamed RS485-B
Other:
- moved on the sheet: U12
Changed lines of the file:
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@@
   (junction (at 103.505 95.885) (diameter 0) (color 0 0 0 0)
   )
+  (junction (at 179.07 94.615) (diameter 0) (color 0 0 0 0)
+  )
   (junction (at 114.935 114.935) (diameter 0) (color 0 0 0 0)
   )
-  (junction (at 172.085 99.695) (diameter 0) (color 0 0 0 0)
+  (junction (at 196.85 99.695) (diameter 0) (color 0 0 0 0)
   )
   (junction (at 142.875 98.425) (diameter 0) (color 0 0 0 0)
@@
   (junction (at 116.205 74.295) (diameter 0) (color 0 0 0 0)
   )
+  (junction (at 179.07 92.075) (diameter 0) (color 0 0 0 0)
+  )
   (wire (pts (xy 128.905 94.615) (xy 138.557 94.615))
     (stroke (width 0) (type default))
@@
     (stroke (width 0) (type default))
   )
+  (wire (pts (xy 176.53 92.075) (xy 179.07 92.075))
+    (stroke (width 0) (type default))
+  )
   (wire (pts (xy 103.505 95.885) (xy 103.505 97.155))
     (stroke (width 0) (type default))
@@
     (stroke (width 0) (type default))
   )
+  (wire (pts (xy 176.53 94.615) (xy 179.07 94.615))
+    (stroke (width 0) (type default))
+  )
   (wire (pts (xy 130.175 99.695) (xy 128.905 99.695))
     (stroke (width 0) (type default))
   )
-  (wire (pts (xy 172.085 86.995) (xy 172.085 99.695))
+  (wire (pts (xy 179.07 86.995) (xy 179.07 92.075))
+    (stroke (width 0) (type default))
+  )
+  (wire (pts (xy 196.85 86.995) (xy 196.85 99.695))
+    (stroke (width 0) (type default))
+  )
+  (wire (pts (xy 179.07 99.695) (xy 179.07 94.615))
     (stroke (width 0) (type default))
   )
@@
     (stroke (width 0) (type default))
   )
-  (wire (pts (xy 172.085 99.695) (xy 172.085 101.6))
+  (wire (pts (xy 196.85 99.695) (xy 196.85 101.6))
     (stroke (width 0) (type default))
   )
@@
     (stroke (width 0) (type default))
   )
-  (wire (pts (xy 155.575 94.615) (xy 160.655 94.615))
+  (wire (pts (xy 178.435 99.695) (xy 179.07 99.695))
     (stroke (width 0) (type default))
   )
@@
     (stroke (width 0) (type default))
   )
-  (wire (pts (xy 160.655 83.185) (xy 160.655 89.535))
+  (wire (pts (xy 179.07 92.075) (xy 185.42 92.075))
+    (stroke (width 0) (type default))
+  )
+  (wire (pts (xy 185.42 83.185) (xy 185.42 89.535))
     (stroke (width 0) (type default))
   )
@@
     (stroke (width 0) (type default))
   )
-  (wire (pts (xy 155.575 92.075) (xy 160.655 92.075))
+  (wire (pts (xy 178.435 86.995) (xy 179.07 86.995))
     (stroke (width 0) (type default))
   )
@@
     (stroke (width 0) (type default))
   )
+  (wire (pts (xy 179.07 94.615) (xy 185.42 94.615))
+    (stroke (width 0) (type default))
+  )
   (wire (pts (xy 129.54 86.36) (xy 129.54 89.535))
     (stroke (width 0) (type default))
@@
     (effects (font (size 1.27 1.27)) (justify right bottom))
   )
-  (label "RS1_A" (at 155.575 92.075 180) (fields_autoplaced)
+  (label "RS1_A" (at 178.435 86.995 180) (fields_autoplaced)
     (effects (font (size 1.27 1.27)) (justify right bottom))
   )
@@
     (effects (font (size 1.27 1.27)) (justify left bottom))
   )
-  (label "RS1_B" (at 155.575 94.615 180) (fields_autoplaced)
+  (label "RS1_B" (at 178.435 99.695 180) (fields_autoplaced)
     (effects (font (size 1.27 1.27)) (justify right bottom))
   )
@@
     (effects (font (size 1.27 1.27)) (justify left bottom))
   )
-  (label "+5V0" (at 160.655 83.185 180) (fields_autoplaced)
+  (label "+5V0" (at 185.42 83.185 180) (fields_autoplaced)
     (effects (font (size 1.27 1.27)) (justify right bottom))
   )
@@
     (effects (font (size 1.27 1.27)) (justify right))
   )
+  (hierarchical_label "RS485-B" (shape input) (at 176.53 94.615 180) (fields_autoplaced)
+    (effects (font (size 1.27 1.27)) (justify right))
+  )
   (hierarchical_label "3V3" (shape input) (at 52.07 80.01 180) (fields_autoplaced)
     (effects (font (size 1.27 1.27)) (justify right))
@@
   )
   (hierarchical_label "GND" (shape input) (at 52.07 84.455 180) (fields_autoplaced)
+    (effects (font (size 1.27 1.27)) (justify right))
+  )
+  (hierarchical_label "RS485-A" (shape input) (at 176.53 92.075 180) (fields_autoplaced)
     (effects (font (size 1.27 1.27)) (justify right))
   )
@@
     )
   )
-  (symbol (lib_id "power:GND") (at 160.655 97.155 0) (mirror y) (unit 1)
-    (in_bom yes) (on_board yes) (dnp no)
-    (property "Reference" "#PWR068" (at 160.655 103.505 0)
-      (effects (font (size 1.27 1.27)) hide)
-    )
-    (property "Value" "GND" (at 157.48 99.06 0)
-      (effects (font (size 1.27 1.27)))
-    )
-    (property "Footprint" "" (at 160.655 97.155 0)
-      (effects (font (size 1.27 1.27)) hide)
-    )
-    (property "Datasheet" "" (at 160.655 97.155 0)
+  (symbol (lib_id "power:GND") (at 185.42 97.155 0) (mirror y) (unit 1)
+    (in_bom yes) (on_board yes) (dnp no)
+    (property "Reference" "#PWR068" (at 185.42 103.505 0)
+      (effects (font (size 1.27 1.27)) hide)
+    )
+    (property "Value" "GND" (at 182.245 99.06 0)
+      (effects (font (size 1.27 1.27)))
+    )
+    (property "Footprint" "" (at 185.42 97.155 0)
+      (effects (font (size 1.27 1.27)) hide)
+    )
+    (property "Datasheet" "" (at 185.42 97.155 0)
       (effects (font (size 1.27 1.27)) hide)
     )
@@
     )
   )
-  (symbol (lib_id "usb-rs485:DF52-4S-0.8H(21)") (at 167.005 93.345 0) (unit 1)
-    (in_bom yes) (on_board yes) (dnp no)
-    (property "Reference" "U12" (at 166.37 81.915 0)
-      (effects (font (size 1.27 1.27)))
-    )
-    (property "Value" "DF52-4S-0.8H(21)" (at 173.355 84.455 0)
-      (effects (font (size 1.27 1.27)))
-    )
-    (property "Footprint" "robot-cortex:DF52-4S-0.8H(21)" (at 169.545 107.315 0)
-      (effects (font (size 1.27 1.27)) hide)
-    )
-    (property "Datasheet" "" (at 169.545 95.885 0)
+  (symbol (lib_id "usb-rs485:DF52-4S-0.8H(21)") (at 191.77 93.345 0) (unit 1)
+    (in_bom yes) (on_board yes) (dnp no)
+    (property "Reference" "U12" (at 191.135 81.915 0)
+      (effects (font (size 1.27 1.27)))
+    )
+    (property "Value" "DF52-4S-0.8H(21)" (at 198.12 84.455 0)
+      (effects (font (size 1.27 1.27)))
+    )
+    (property "Footprint" "robot-cortex:DF52-4S-0.8H(21)" (at 194.31 107.315 0)
+      (effects (font (size 1.27 1.27)) hide)
+    )
+    (property "Datasheet" "" (at 194.31 95.885 0)
       (effects (font (size 1.27 1.27)) hide)
     )
@@
     )
   )
-  (symbol (lib_id "power:GND") (at 172.085 101.6 0) (mirror y) (unit 1)
-    (in_bom yes) (on_board yes) (dnp no)
-    (property "Reference" "#PWR069" (at 172.085 107.95 0)
-      (effects (font (size 1.27 1.27)) hide)
-    )
-    (property "Value" "GND" (at 168.91 103.505 0)
-      (effects (font (size 1.27 1.27)))
-    )
-    (property "Footprint" "" (at 172.085 101.6 0)
-      (effects (font (size 1.27 1.27)) hide)
-    )
-    (property "Datasheet" "" (at 172.085 101.6 0)
-      (effects (font (size 1.27 1.27)) hide)
-    )
+  (symbol (lib_id "power:GND") (at 196.85 101.6 0) (mirror y) (unit 1)
+    (in_bom yes) (on_board yes) (dnp no)
+    (property "Reference" "#PWR069" (at 196.85 107.95 0)
+      (effects (font (size 1.27 1.27)) hide)
+    )
+    (property "Value" "GND" (at 193.675 103.505 0)
+      (effects (font (size 1.27 1.27)))
+    )
+    (property "Footprint" "" (at 196.85 101.6 0)
+      (effects (font (size 1.27 1.27)) hide)
+    )
+    (property "Datasheet" "" (at 196.85 101.6 0)
+      (effects (font (size 1.27 1.27)) hide)
+    )

Commit message: rename library to be for this
Parts:
- C9: footprint robot-cortex:C_0603_1608Metric -> usb-rs485:C_0603_1608Metric
- IC1: footprint robot-cortex:THVD2410VDRCR -> usb-rs485:THVD2410VDRCR
- R19: footprint robot-cortex:R_0402_1005Metric -> usb-rs485:R_0402_1005Metric
- U12: footprint robot-cortex:DF52-4S-0.8H(21) -> usb-rs485:DF52-4S-0.8H(21)
Changed lines of the file:
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@@
       (effects (font (size 1.27 1.27)) (justify left))
     )
-    (property "Footprint" "robot-cortex:THVD2410VDRCR" (at 125.095 176.835 0)
+    (property "Footprint" "usb-rs485:THVD2410VDRCR" (at 125.095 176.835 0)
       (effects (font (size 1.27 1.27)) (justify left top) hide)
     )
@@
       (effects (font (size 1.27 1.27)) (justify left))
     )
-    (property "Footprint" "robot-cortex:C_0603_1608Metric" (at 148.8948 66.675 0)
+    (property "Footprint" "usb-rs485:C_0603_1608Metric" (at 148.8948 66.675 0)
       (effects (font (size 1.27 1.27)) hide)
     )
@@
       (effects (font (size 1.27 1.27)))
     )
-    (property "Footprint" "robot-cortex:DF52-4S-0.8H(21)" (at 194.31 107.315 0)
+    (property "Footprint" "usb-rs485:DF52-4S-0.8H(21)" (at 194.31 107.315 0)
       (effects (font (size 1.27 1.27)) hide)
     )
@@
       (effects (font (size 1.27 1.27)))
     )
-    (property "Footprint" "robot-cortex:R_0402_1005Metric" (at 137.795 106.045 0)
-      (effects (font (size 1.27 1.27)) hide)
-    )
+    (property "Footprint" "usb-rs485:R_0402_1005Metric" (at 137.795 106.045 0)
+      (effects (font (size 1.27 1.27)) hide)
+    )

Commit message: moved it elsewhere but MEH
Connections:
- net 5V0: no longer U12.1
- new net VLOGIC_MOTOR: U12.1
Changed lines of the file:
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@@
     (stroke (width 0) (type default))
   )
-  (wire (pts (xy 185.42 83.185) (xy 185.42 89.535))
+  (wire (pts (xy 185.42 80.01) (xy 185.42 89.535))
     (stroke (width 0) (type default))
   )
@@
     (effects (font (size 1.27 1.27)) (justify left bottom))
   )
-  (label "+5V0" (at 185.42 83.185 180) (fields_autoplaced)
-    (effects (font (size 1.27 1.27)) (justify right bottom))
-  )
   (hierarchical_label "UART_TX" (shape input) (at 52.07 93.345 180) (fields_autoplaced)
     (effects (font (size 1.27 1.27)) (justify right))
@@
     (effects (font (size 1.27 1.27)) (justify right))
   )
+  (hierarchical_label "VLOGIC_MOTOR" (shape input) (at 185.42 80.01 180) (fields_autoplaced)
+    (effects (font (size 1.27 1.27)) (justify right))
+  )
